File: Danck.kicad_pcb (KiCad board)
At the start: 2 copper layers, 98 parts, among them U1 ProMicro

Commit message: row 3 is in
Parts:
- moved MX36 289.8 mm to (247.7, 76.2)
- moved MX35 270.8 mm to (228.6, 76.2)
- moved MX34 251.7 mm to (209.6, 76.2)
- moved MX33 232.7 mm to (190.5, 76.2)
- moved MX32 213.7 mm to (171.4, 76.2)
- moved MX31 194.6 mm to (152.4, 76.2)
- moved MX30 175.6 mm to (133.3, 76.2)
- moved MX29 156.6 mm to (114.3, 76.2)
- moved MX28 137.6 mm to (95.2, 76.2)
- moved MX27 118.6 mm to (76.2, 76.2)
- moved MX26 99.6 mm to (57.1, 76.2)
- moved MX25 80.6 mm to (38.1, 76.2)
Changed lines of the file:
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@@
   )
   (module MX_Alps_Hybrid:MX-1U-NoLED (layer F.Cu)
-    (at -41.9989 66.9036)
+    (at 38.1 76.2)
     (fp_text reference MX25 (at 0 3.175) (layer F.SilkS)
       (effects (font (size 1 1) (thickness 0.15)))
@@
   )
   (module MX_Alps_Hybrid:MX-1U-NoLED (layer F.Cu)
-    (at -41.9989 66.9036)
+    (at 57.15 76.2)
     (fp_text reference MX26 (at 0 3.175) (layer F.SilkS)
       (effects (font (size 1 1) (thickness 0.15)))
@@
   )
   (module MX_Alps_Hybrid:MX-1U-NoLED (layer F.Cu)
-    (at -41.9989 66.9036)
+    (at 76.2 76.2)
     (fp_text reference MX27 (at 0 3.175) (layer F.SilkS)
       (effects (font (size 1 1) (thickness 0.15)))
@@
   )
   (module MX_Alps_Hybrid:MX-1U-NoLED (layer F.Cu)
-    (at -41.9989 66.9036)
+    (at 95.25 76.2)
     (fp_text reference MX28 (at 0 3.175) (layer F.SilkS)
       (effects (font (size 1 1) (thickness 0.15)))
@@
   )
   (module MX_Alps_Hybrid:MX-1U-NoLED (layer F.Cu)
-    (at -41.9989 66.9036)
+    (at 114.3 76.2)
     (fp_text reference MX29 (at 0 3.175) (layer F.SilkS)
       (effects (font (size 1 1) (thickness 0.15)))
@@
   )
   (module MX_Alps_Hybrid:MX-1U-NoLED (layer F.Cu)
-    (at -41.9989 66.9036)
+    (at 133.35 76.2)
     (fp_text reference MX30 (at 0 3.175) (layer F.SilkS)
       (effects (font (size 1 1) (thickness 0.15)))
@@
   )
   (module MX_Alps_Hybrid:MX-1U-NoLED (layer F.Cu)
-    (at -41.9989 66.9036)
+    (at 152.4 76.2)
     (fp_text reference MX31 (at 0 3.175) (layer F.SilkS)
       (effects (font (size 1 1) (thickness 0.15)))
@@
   )
   (module MX_Alps_Hybrid:MX-1U-NoLED (layer F.Cu)
-    (at -41.9989 66.9036)
+    (at 171.45 76.2)
     (fp_text reference MX32 (at 0 3.175) (layer F.SilkS)
       (effects (font (size 1 1) (thickness 0.15)))
@@
   )
   (module MX_Alps_Hybrid:MX-1U-NoLED (layer F.Cu)
-    (at -41.9989 66.9036)
+    (at 190.5 76.2)
     (fp_text reference MX33 (at 0 3.175) (layer F.SilkS)
       (effects (font (size 1 1) (thickness 0.15)))
@@
   )
   (module MX_Alps_Hybrid:MX-1U-NoLED (layer F.Cu)
-    (at -41.9989 66.9036)
+    (at 209.55 76.2)
     (fp_text reference MX34 (at 0 3.175) (layer F.SilkS)
       (effects (font (size 1 1) (thickness 0.15)))
@@
   )
   (module MX_Alps_Hybrid:MX-1U-NoLED (layer F.Cu)
-    (at -41.9989 66.9036)
+    (at 228.6 76.2)
     (fp_text reference MX35 (at 0 3.175) (layer F.SilkS)
       (effects (font (size 1 1) (thickness 0.15)))
@@
   )
   (module MX_Alps_Hybrid:MX-1U-NoLED (layer F.Cu)
-    (at -41.9989 66.9036)
+    (at 247.65 76.2)
     (fp_text reference MX36 (at 0 3.175) (layer F.SilkS)
       (effects (font (size 1 1) (thickness 0.15)))

Commit message: Finish grid
Parts:
- moved MX48 291.0 mm to (247.7, 95.2)
- moved MX47 272.1 mm to (228.6, 95.2)
- moved MX46 253.1 mm to (209.6, 95.2)
- moved MX45 234.2 mm to (190.5, 95.2)
- moved MX44 215.3 mm to (171.4, 95.2)
- moved MX43 196.5 mm to (152.4, 95.2)
- moved MX49 187.0 mm to (142.9, 95.2)
- moved MX42 177.6 mm to (133.3, 95.2)
- moved MX41 158.8 mm to (114.3, 95.2)
- moved MX40 140.1 mm to (95.2, 95.2)
- moved MX39 121.6 mm to (76.2, 95.2)
- moved MX38 103.1 mm to (57.1, 95.2)
- moved MX37 85.0 mm to (38.1, 95.2)
Changed lines of the file:
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@@
   )
   (module MX_Alps_Hybrid:MX-1U-NoLED (layer F.Cu)
-    (at -41.9989 66.9036)
+    (at 38.1 95.25)
     (fp_text reference MX37 (at 0 3.175) (layer F.SilkS)
       (effects (font (size 1 1) (thickness 0.15)))
@@
   )
   (module MX_Alps_Hybrid:MX-1U-NoLED (layer F.Cu)
-    (at -41.9989 66.9036)
+    (at 57.15 95.25)
     (fp_text reference MX38 (at 0 3.175) (layer F.SilkS)
       (effects (font (size 1 1) (thickness 0.15)))
@@
   )
   (module MX_Alps_Hybrid:MX-1U-NoLED (layer F.Cu)
-    (at -41.9989 66.9036)
+    (at 76.2 95.25)
     (fp_text reference MX39 (at 0 3.175) (layer F.SilkS)
       (effects (font (size 1 1) (thickness 0.15)))
@@
   )
   (module MX_Alps_Hybrid:MX-1U-NoLED (layer F.Cu)
-    (at -41.9989 66.9036)
+    (at 95.25 95.25)
     (fp_text reference MX40 (at 0 3.175) (layer F.SilkS)
       (effects (font (size 1 1) (thickness 0.15)))
@@
   )
   (module MX_Alps_Hybrid:MX-1U-NoLED (layer F.Cu)
-    (at -41.9989 66.9036)
+    (at 114.3 95.25)
     (fp_text reference MX41 (at 0 3.175) (layer F.SilkS)
       (effects (font (size 1 1) (thickness 0.15)))
@@
   )
   (module MX_Alps_Hybrid:MX-1U-NoLED (layer F.Cu)
-    (at -41.9989 66.9036)
+    (at 133.35 95.25)
     (fp_text reference MX42 (at 0 3.175) (layer F.SilkS)
       (effects (font (size 1 1) (thickness 0.15)))
@@
   )
   (module MX_Alps_Hybrid:MX-1U-NoLED (layer F.Cu)
-    (at -41.9989 66.9036)
+    (at 152.4 95.25)
     (fp_text reference MX43 (at 0 3.175) (layer F.SilkS)
       (effects (font (size 1 1) (thickness 0.15)))
@@
   )
   (module MX_Alps_Hybrid:MX-1U-NoLED (layer F.Cu)
-    (at -41.9989 66.9036)
+    (at 171.45 95.25)
     (fp_text reference MX44 (at 0 3.175) (layer F.SilkS)
       (effects (font (size 1 1) (thickness 0.15)))
@@
   )
   (module MX_Alps_Hybrid:MX-1U-NoLED (layer F.Cu)
-    (at -41.9989 66.9036)
+    (at 190.5 95.25)
     (fp_text reference MX45 (at 0 3.175) (layer F.SilkS)
       (effects (font (size 1 1) (thickness 0.15)))
@@
   )
   (module MX_Alps_Hybrid:MX-1U-NoLED (layer F.Cu)
-    (at -41.9989 66.9036)
+    (at 209.55 95.25)
     (fp_text reference MX46 (at 0 3.175) (layer F.SilkS)
       (effects (font (size 1 1) (thickness 0.15)))
@@
   )
   (module MX_Alps_Hybrid:MX-1U-NoLED (layer F.Cu)
-    (at -41.9989 66.9036)
+    (at 228.6 95.25)
     (fp_text reference MX47 (at 0 3.175) (layer F.SilkS)
       (effects (font (size 1 1) (thickness 0.15)))
@@
   )
   (module MX_Alps_Hybrid:MX-1U-NoLED (layer F.Cu)
-    (at -41.9989 66.9036)
+    (at 247.65 95.25)
     (fp_text reference MX48 (at 0 3.175) (layer F.SilkS)
       (effects (font (size 1 1) (thickness 0.15)))
@@
   )
   (module MX_Alps_Hybrid:MX-2U-ReversedStabilizers-NoLED (layer F.Cu)
-    (at -41.9989 66.9036)
+    (at 142.875 95.25)
     (fp_text reference MX49 (at 0 3.175) (layer F.SilkS)
       (effects (font (size 1 1) (thickness 0.15)))

Commit message: Finish the dank memes
Parts:
- added G***: LOGO, memelogo:snoopdogg, B.Cu at (85.7, 46.8)
- added G***: LOGO, memelogo:cartel, F.Cu at (100.0, 66.7)
- added G***: LOGO, memelogo:danck, F.Cu at (167.5, 66.7)
- added G***: LOGO, ai03-logo:AI03-Silkscreen-5.4mm-Text, F.Cu at (127.8, 66.7)
- added G***: LOGO, memelogo:dickbutt, B.Cu at (50.0, 74.6)
- added G***: LOGO, memelogo:assdropfixed, B.Cu at (221.5, 84.1)
- added G***: LOGO, memelogo:reesrlarge, B.Cu at (117.5, 82.5)
- added G***: LOGO, memelogo:bobbyhill, B.Cu at (181.0, 83.8)
- added G***: LOGO, memelogo:bobox, B.Cu at (156.4, 69.5)
- added G***: LOGO, memelogo:datboi, B.Cu at (105.6, 54.0)
- added G***: LOGO, memelogo:thonk, B.Cu at (77.0, 88.1)
- added G***: LOGO, memelogo:thinkster, B.Cu at (127.8, 62.7)
- added REF**: mountinghole, locallib:mountinghole, F.Cu at (142.9, 66.7)
- added REF**: mountinghole, locallib:mountinghole, F.Cu at (238.1, 85.7)
- added REF**: mountinghole, locallib:mountinghole, F.Cu at (47.6, 85.7)
- added REF**: mountinghole, locallib:mountinghole, F.Cu at (200.0, 47.6)
- added REF**: mountinghole, locallib:mountinghole, F.Cu at (85.7, 47.6)
- added SW1: SW_PUSH, Molex-0548190589:PushButton_6x6mm_TH, B.Cu at (66.7, 85.7)
- U1: moved to B.Cu
- moved D12 293.9 mm to (251.3, 47.6), turned to 180 degrees
- moved D48 293.9 mm to (251.3, 85.7), turned to 180 degrees
- moved D24 293.3 mm to (251.3, 66.7), turned to 180 degrees
- moved D47 281.9 mm to (238.1, 98.9), turned to 90 degrees
- moved D11 281.3 mm to (238.1, 41.8), turned to 90 degrees
- moved D36 280.4 mm to (238.1, 79.9), turned to 90 degrees
- moved D23 280.2 mm to (238.1, 60.8), turned to 90 degrees
- moved D35 274.9 mm to (232.3, 85.7), turned to 180 degrees
- moved D46 263.0 mm to (219.1, 98.9), turned to 90 degrees
- moved D10 262.3 mm to (219.1, 41.8), turned to 90 degrees
- moved D34 261.4 mm to (219.1, 79.9), turned to 90 degrees
- moved D22 261.1 mm to (219.1, 60.8), turned to 90 degrees
- moved D45 244.1 mm to (200.0, 98.9), turned to 90 degrees
- moved D9 243.3 mm to (200.0, 41.8), turned to 90 degrees
- moved D33 242.4 mm to (200.0, 79.9), turned to 90 degrees
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Connections:
- net Net-(U1-Pad21) renamed +5V
- U1 pad 1: Net-(U1-Pad1) -> COL11
- U1 pad 10: Net-(U1-Pad10) -> COL4
- U1 pad 11: Net-(U1-Pad11) -> COL3
- U1 pad 12: Net-(U1-Pad12) -> COL2
- U1 pad 13: Net-(U1-Pad13) -> ROW3
- U1 pad 14: Net-(U1-Pad14) -> ROW2
- U1 pad 15: Net-(U1-Pad15) -> ROW1
- U1 pad 18: Net-(U1-Pad18) -> ROW0
- U1 pad 19: Net-(U1-Pad19) -> COL1
- U1 pad 2: Net-(U1-Pad2) -> COL10
- U1 pad 20: Net-(U1-Pad20) -> COL0
- U1 pad 23: Net-(U1-Pad23) -> GND
- U1 pad 3: Net-(U1-Pad3) -> GND
- U1 pad 4: Net-(U1-Pad4) -> GND
- U1 pad 5: Net-(U1-Pad5) -> COL9
- U1 pad 6: Net-(U1-Pad6) -> COL8
- U1 pad 7: Net-(U1-Pad7) -> COL7
- U1 pad 8: Net-(U1-Pad8) -> COL6
- U1 pad 9: Net-(U1-Pad9) -> COL5
Routing:
- net ROW0: track 0.00 -> 278.3 mm
- net ROW3: track 0.00 -> 261.1 mm
- net COL11: track 0.00 -> 251.5 mm
- net ROW1: track 0.00 -> 240.5 mm
- net COL10: track 0.00 -> 232.4 mm
- net ROW2: track 0.00 -> 222.4 mm
- net COL9: track 0.00 -> 208.9 mm
- net COL8: track 0.00 -> 185.3 mm
- net COL7: track 0.00 -> 165.8 mm
- net COL6: track 0.00 -> 147.8 mm
- net COL5: track 0.00 -> 142.9 mm
- net COL4: track 0.00 -> 114.6 mm
- net COL3: track 0.00 -> 93.5 mm
- net COL0: track 0.00 -> 78.2 mm
- net GND: track 0.00 -> 73.0 mm
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- added copper zone on B.Cu, net GND
- added copper zone on F.Cu, net GND
Other:
- board outline added: 228.6 x 76.2 mm
- board text added: "+5V"
- board text added: "DANCK"
- board text added: "Extremely low-cost Ortholinear keyboard"
- board text added: "Hella cheap ortho"
