File: Danck.kicad_pcb (KiCad board)
At the start: 2 copper layers, 228.6 x 76.2 mm, 123 parts, among them P1 Pad, P2 Pad, P3 Pad, P4 Pad, SW1 SW_PUSH, U1 ProMicro

Commit message: Add memes and update gerber
Parts:
- added G***: LOGO, memelogo:magicalleaf, B.Cu at (241.6, 90.2)
- added G***: LOGO, memelogo:dopre, B.Cu at (82.9, 89.6)
- moved G*** 8.42 mm to (65.2, 89.2)
Other:
- board text added: "CAUTION Toxic Memes DO NOT EAT"
