File: Danck.sch (KiCad schematic (older format))
At the start: 1 part

Commit message: Finish schematic
Well... that was fast
Parts:
- added D1, D10, D11, D12, D13, D14, D15, D16, D17, D18, D19, D2, D20, D21, D22, D23, D24, D25, D26, D27, D28, D29, D3, D30, D31, D32, D33, D34, D35, D36, D37, D38, D39, D4, D40, D41, D42, D43, D44, D45, D46, D47, D48, D5, D6, D7, D8, D9: 1N4148, Diodes_THT:D_DO-35_SOD27_P7.62mm_Horizontal, symbol D_Small
- added MX1, MX10, MX11, MX12, MX13, MX14, MX15, MX16, MX17, MX18, MX19, MX2, MX20, MX21, MX22, MX23, MX24, MX25, MX26, MX27, MX28, MX29, MX3, MX30, MX31, MX32, MX33, MX34, MX35, MX36, MX37, MX38, MX39, MX4, MX40, MX41, MX42, MX43, MX44, MX45, MX46, MX47, MX48, MX5, MX6, MX7, MX8, MX9: MX-1U, MX_Alps_Hybrid:MX-1U-NoLED, symbol MX-1U
- added MX49: MX-2U, MX_Alps_Hybrid:MX-2U-ReversedStabilizers-NoLED, symbol MX-2U
- U1: renamed from U?; footprint (none) -> locallib:pro_micro
Connections:
- new net: D1.2 (A), MX1.2 (ROW)
- new net: D2.2 (A), MX2.2 (ROW)
- new net: D3.2 (A), MX3.2 (ROW)
- new net: D4.2 (A), MX4.2 (ROW)
- new net: D5.2 (A), MX5.2 (ROW)
- new net: D6.2 (A), MX6.2 (ROW)
- new net: D7.2 (A), MX7.2 (ROW)
- new net: D8.2 (A), MX8.2 (ROW)
- new net: D9.2 (A), MX9.2 (ROW)
- new net: D10.2 (A), MX10.2 (ROW)
- new net: D11.2 (A), MX11.2 (ROW)
- new net: D12.2 (A), MX12.2 (ROW)
- new net: D13.2 (A), MX13.2 (ROW)
- new net: D14.2 (A), MX14.2 (ROW)
- new net: D15.2 (A), MX15.2 (ROW)
- new net: D16.2 (A), MX16.2 (ROW)
- new net: D17.2 (A), MX17.2 (ROW)
- new net: D18.2 (A), MX18.2 (ROW)
- new net: D19.2 (A), MX19.2 (ROW)
- new net: D20.2 (A), MX20.2 (ROW)
- new net: D21.2 (A), MX21.2 (ROW)
- new net: D22.2 (A), MX22.2 (ROW)
- new net: D23.2 (A), MX23.2 (ROW)
- new net: D24.2 (A), MX24.2 (ROW)
- new net: D25.2 (A), MX25.2 (ROW)
- new net: D26.2 (A), MX26.2 (ROW)
- new net: D27.2 (A), MX27.2 (ROW)
- new net: D28.2 (A), MX28.2 (ROW)
- new net: D29.2 (A), MX29.2 (ROW)
- new net: D30.2 (A), MX30.2 (ROW)
- new net: D31.2 (A), MX31.2 (ROW)
- new net: D32.2 (A), MX32.2 (ROW)
- new net: D33.2 (A), MX33.2 (ROW)
- new net: D34.2 (A), MX34.2 (ROW)
- new net: D35.2 (A), MX35.2 (ROW)
- new net: D36.2 (A), MX36.2 (ROW)
- new net: D37.2 (A), MX37.2 (ROW)
- new net: D38.2 (A), MX38.2 (ROW)
- new net: D39.2 (A), MX39.2 (ROW)
- new net: D40.2 (A), MX40.2 (ROW)
- new net: D41.2 (A), MX41.2 (ROW)
- new net: D42.2 (A), MX42.2 (ROW), MX49.2 (ROW)
- new net: D43.2 (A), MX43.2 (ROW)
- new net: D44.2 (A), MX44.2 (ROW)
- new net: D45.2 (A), MX45.2 (ROW)
- new net: D46.2 (A), MX46.2 (ROW)
- new net: D47.2 (A), MX47.2 (ROW)
- new net: D48.2 (A), MX48.2 (ROW)
- new net COL0: MX1.1 (COL), MX13.1 (COL), MX25.1 (COL), MX37.1 (COL)
- new net COL1: MX14.1 (COL), MX2.1 (COL), MX26.1 (COL), MX38.1 (COL)
- new net COL10: MX11.1 (COL), MX23.1 (COL), MX35.1 (COL), MX47.1 (COL)
- new net COL11: MX12.1 (COL), MX24.1 (COL), MX36.1 (COL), MX48.1 (COL)
- new net COL2: MX15.1 (COL), MX27.1 (COL), MX3.1 (COL), MX39.1 (COL)
- new net COL3: MX16.1 (COL), MX28.1 (COL), MX4.1 (COL), MX40.1 (COL)
- new net COL4: MX17.1 (COL), MX29.1 (COL), MX41.1 (COL), MX5.1 (COL)
- new net COL5: MX18.1 (COL), MX30.1 (COL), MX42.1 (COL), MX49.1 (COL), MX6.1 (COL)
- new net COL6: MX19.1 (COL), MX31.1 (COL), MX43.1 (COL), MX7.1 (COL)
- new net COL7: MX20.1 (COL), MX32.1 (COL), MX44.1 (COL), MX8.1 (COL)
- new net COL8: MX21.1 (COL), MX33.1 (COL), MX45.1 (COL), MX9.1 (COL)
- new net COL9: MX10.1 (COL), MX22.1 (COL), MX34.1 (COL), MX46.1 (COL)
- new net ROW0: D1.1 (K), D10.1 (K), D11.1 (K), D12.1 (K), D2.1 (K), D3.1 (K), D4.1 (K), D5.1 (K), D6.1 (K), D7.1 (K), D8.1 (K), D9.1 (K)
- new net ROW1: D13.1 (K), D14.1 (K), D15.1 (K), D16.1 (K), D17.1 (K), D18.1 (K), D19.1 (K), D20.1 (K), D21.1 (K), D22.1 (K), D23.1 (K), D24.1 (K)
- new net ROW2: D25.1 (K), D26.1 (K), D27.1 (K), D28.1 (K), D29.1 (K), D30.1 (K), D31.1 (K), D32.1 (K), D33.1 (K), D34.1 (K), D35.1 (K), D36.1 (K)
- new net ROW3: D37.1 (K), D38.1 (K), D39.1 (K), D40.1 (K), D41.1 (K), D42.1 (K), D43.1 (K), D44.1 (K), D45.1 (K), D46.1 (K), D47.1 (K), D48.1 (K)

Commit message: Finish the dank memes
Parts:
- added SW1: SW_PUSH, Molex-0548190589:PushButton_6x6mm_TH, symbol SW_PUSH
Connections:
- net COL0: now also U1.20 (21)
- net COL1: now also U1.19 (20)
- net COL10: now also U1.2 (0)
- net COL11: now also U1.1
- net COL2: now also U1.12 (9)
- net COL3: now also U1.11 (8)
- net COL4: now also U1.10 (7)
- net COL5: now also U1.9 (6)
- net COL6: now also U1.8 (5)
- net COL7: now also U1.7 (4)
- net COL8: now also U1.6 (3)
- net COL9: now also U1.5 (2)
- net ROW0: now also U1.18 (19)
- net ROW1: now also U1.15 (14)
- net ROW2: now also U1.14 (16)
- net ROW3: now also U1.13 (10)
- net +5V: now reaches U1.21 (5V)
- net at U1.22 (RST): now also SW1.1
- net GND: now reaches U1.23 (GND)
- net GND: now also U1.3 (GND), U1.4 (GND), SW1.2
Changed lines of the file:
@@
 LIBS:Molex-0548190589
 LIBS:MX_Alps_Hybrids
+LIBS:Danck-cache
 EELAYER 25 0
 EELAYER END
@@
 Wire Wire Line
 	6025 5000 6175 5000
+$Comp
+L GND #PWR01
+U 1 1 5A2BAA24
+P 850 1050
+F 0 "#PWR01" H 850 800 50  0001 C CNN
+F 1 "GND" H 850 900 50  0000 C CNN
+F 2 "" H 850 1050 50  0001 C CNN
+F 3 "" H 850 1050 50  0001 C CNN
+	1    850  1050
+	0    1    1    0
+$EndComp
+$Comp
+L GND #PWR02
+U 1 1 5A2BAAFC
+P 850 1150
+F 0 "#PWR02" H 850 900 50  0001 C CNN
+F 1 "GND" H 850 1000 50  0000 C CNN
+F 2 "" H 850 1150 50  0001 C CNN
+F 3 "" H 850 1150 50  0001 C CNN
+	1    850  1150
+	0    1    1    0
+$EndComp
+$Comp
+L GND #PWR03
+U 1 1 5A2BABD4
+P 1750 950
+F 0 "#PWR03" H 1750 700 50  0001 C CNN
+F 1 "GND" H 1750 800 50  0000 C CNN
+F 2 "" H 1750 950 50  0001 C CNN
+F 3 "" H 1750 950 50  0001 C CNN
+	1    1750 950
+	0    -1   -1   0
+$EndComp
+$Comp
+L SW_PUSH SW1
+U 1 1 5A2BAD84
+P 2050 1050
+F 0 "SW1" H 2200 1160 50  0000 C CNN
+F 1 "SW_PUSH" H 2050 970 50  0000 C CNN
+F 2 "Molex-0548190589:PushButton_6x6mm_TH" H 2050 1050 60  0001 C CNN
+F 3 "" H 2050 1050 60  0000 C CNN
+	1    2050 1050
+	1    0    0    -1
+$EndComp
+$Comp
+L GND #PWR04
+U 1 1 5A2BAE73
+P 2350 1050
+F 0 "#PWR04" H 2350 800 50  0001 C CNN
+F 1 "GND" H 2350 900 50  0000 C CNN
+F 2 "" H 2350 1050 50  0001 C CNN
+F 3 "" H 2350 1050 50  0001 C CNN
+	1    2350 1050
+	0    -1   -1   0
+$EndComp
+$Comp
+L +5V #PWR05
+U 1 1 5A2BD3A9
+P 1750 1150
+F 0 "#PWR05" H 1750 1000 50  0001 C CNN
+F 1 "+5V" H 1750 1290 50  0000 C CNN
+F 2 "" H 1750 1150 50  0001 C CNN
+F 3 "" H 1750 1150 50  0001 C CNN
+	1    1750 1150
+	0    1    1    0
+$EndComp
+Text GLabel 850  850  0    60   Input ~ 0
+COL11
+Text GLabel 850  950  0    60   Input ~ 0
+COL10
+Text GLabel 850  1250 0    60   Input ~ 0
+COL9
+Text GLabel 850  1350 0    60   Input ~ 0
+COL8
+Text GLabel 850  1450 0    60   Input ~ 0
+COL7
+Text GLabel 850  1550 0    60   Input ~ 0
+COL6
+Text GLabel 850  1750 0    60   Input ~ 0
+COL4
+Text GLabel 850  1650 0    60   Input ~ 0
+COL5
+Text GLabel 850  1850 0    60   Input ~ 0
+COL3
+Text GLabel 850  1950 0    60   Input ~ 0
+COL2
+Text GLabel 1750 1250 2    60   Input ~ 0
+COL0
+Text GLabel 1750 1350 2    60   Input ~ 0
+COL1
+Text GLabel 1750 1950 2    60   Input ~ 0
+ROW3
+Text GLabel 1750 1850 2    60   Input ~ 0
+ROW2
+Text GLabel 1750 1750 2    60   Input ~ 0
+ROW1
+Text GLabel 1750 1450 2    60   Input ~ 0
+ROW0
 $EndSCHEMATC

Commit message: breakout pins
Parts:
- added P1, P2, P3, P4: Pad, locallib:mountinghole, symbol R
Connections:
- net +5V: now also P3.1
- net GND: now also P4.1
- net at U1.16 (15): now also P2.1
- net at U1.17 (18): now also P1.1
Changed lines of the file:
@@
 Text GLabel 1750 1450 2    60   Input ~ 0
 ROW0
+$Comp
+L R P1
+U 1 1 5A322ABB
+P 2450 1550
+F 0 "P1" V 2530 1550 50  0000 C CNN
+F 1 "Pad" V 2450 1550 50  0000 C CNN
+F 2 "locallib:mountinghole" V 2380 1550 50  0001 C CNN
+F 3 "" H 2450 1550 50  0001 C CNN
+	1    2450 1550
+	0    -1   -1   0
+$EndComp
+$Comp
+L R P2
+U 1 1 5A322DD0
+P 2450 1725
+F 0 "P2" V 2530 1725 50  0000 C CNN
+F 1 "Pad" V 2450 1725 50  0000 C CNN
+F 2 "locallib:mountinghole" V 2380 1725 50  0001 C CNN
+F 3 "" H 2450 1725 50  0001 C CNN
+	1    2450 1725
+	0    -1   -1   0
+$EndComp
+Wire Wire Line
+	2300 1550 1750 1550
+Wire Wire Line
+	1750 1650 2300 1650
+Wire Wire Line
+	2300 1650 2300 1725
+$Comp
+L R P3
+U 1 1 5A323624
+P 2450 1900
+F 0 "P3" V 2530 1900 50  0000 C CNN
+F 1 "Pad" V 2450 1900 50  0000 C CNN
+F 2 "locallib:mountinghole" V 2380 1900 50  0001 C CNN
+F 3 "" H 2450 1900 50  0001 C CNN
+	1    2450 1900
+	0    -1   -1   0
+$EndComp
+$Comp
+L +5V #PWR06
+U 1 1 5A323A72
+P 2300 1900
+F 0 "#PWR06" H 2300 1750 50  0001 C CNN
+F 1 "+5V" H 2300 2040 50  0000 C CNN
+F 2 "" H 2300 1900 50  0001 C CNN
+F 3 "" H 2300 1900 50  0001 C CNN
+	1    2300 1900
+	0    -1   -1   0
+$EndComp
+$Comp
+L R P4
+U 1 1 5A323BB6
+P 2450 2075
+F 0 "P4" V 2530 2075 50  0000 C CNN
+F 1 "Pad" V 2450 2075 50  0000 C CNN
+F 2 "locallib:mountinghole" V 2380 2075 50  0001 C CNN
+F 3 "" H 2450 2075 50  0001 C CNN
+	1    2450 2075
+	0    -1   -1   0
+$EndComp
+$Comp
+L GND #PWR07
+U 1 1 5A323E4A
+P 2300 2075
+F 0 "#PWR07" H 2300 1825 50  0001 C CNN
+F 1 "GND" H 2300 1925 50  0000 C CNN
+F 2 "" H 2300 2075 50  0001 C CNN
+F 3 "" H 2300 2075 50  0001 C CNN
+	1    2300 2075
+	0    1    1    0
+$EndComp
 $EndSCHEMATC
