File: Contra.kicad_pcb (KiCad board)
At the start: 2 copper layers, 231 x 76.2 mm, 111 parts, among them P1 Pad, P2 Pad, P3 Pad, P4 Pad, SW1 SW_PUSH, U1 ProMicro

Commit message: Revert "Unroute, prepare for reroute"
This reverts commit 2692a349e5744fa5fd6682816f15a667edd49ab0.
Parts:
- added G***: LOGO, memelogo:wey, B.Cu at (43.6, 51.9)
- added G***: LOGO, memelogo:boboxsmall, B.Cu at (45.7, 87.6)
- added G***: LOGO, memelogo:thonksmall, B.Cu at (134.6, 53.3)
- added G***: LOGO, memelogo:thinkster, B.Cu at (71.1, 86.4)
- added G***: LOGO, memelogo:datboi, B.Cu at (90.2, 71.1)
- added G***: LOGO, memelogo:bobbyhill, B.Cu at (218.4, 84.7)
- added G***: LOGO, memelogo:dickbutt, B.Cu at (102.6, 85.3)
- added G***: LOGO, memelogo:broken, B.Cu at (186.9, 82.2)
- added G***: LOGO, memelogo:youwat, B.Cu at (160.0, 67.3)
- added G***: LOGO, memelogo:dopre, B.Cu at (108.0, 58.4)
- added G***: LOGO, memelogo:magicalleaf, B.Cu at (241.6, 90.2)
- added G***: LOGO, memelogo:reeeeeee, B.Cu at (221.5, 47.6)
- added G***: LOGO, memelogo:stem, B.Cu at (61.5, 62.9)
- added G***: LOGO, memelogo:righthand, B.Cu at (141.4, 82.4)
Routing:
- net ROW0: track 0.00 -> 270.5 mm
- net ROW3: track 0.00 -> 269.8 mm
- net ROW1: track 0.00 -> 232.7 mm
- net COL11: track 0.00 -> 232.1 mm
- net ROW2: track 0.00 -> 222.0 mm
- net COL10: track 0.00 -> 212.9 mm
- net COL9: track 0.00 -> 184.7 mm
- net COL8: track 0.00 -> 164.6 mm
- net COL7: track 0.00 -> 145.4 mm
- net COL6: track 0.00 -> 127.0 mm
- net COL5: track 0.00 -> 120.3 mm
- net COL0: track 0.00 -> 105.3 mm
- net COL4: track 0.00 -> 93.9 mm
- net GND: track 0.00 -> 93.6 mm
- net +5V: track 0.00 -> 77.4 mm, vias 0 -> 1
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- added copper zone on B.Cu, net GND
- added copper zone on F.Cu, net GND
Other:
- net class Default: trace_width 0.254 -> 0.25
- net class Power removed
- board text added: "+5V"
- board text added: "CAUTION: Toxic Memes. DO NOT EAT. Do not wash with beer."
- board text added: "CONTRA"
- board text added: "Pro Micro here! Component side faces away from the PCB. Rev 1.6"
- board text added: "criminally cheap ortho"
- board text removed: "Pro Micro here! Component side faces away from the PCB. Rev 2.0"

Commit message: Opt to reroute instead of rebuild from scratch
Parts:
- removed the G*** at (43.6, 51.9)
- removed the G*** at (45.7, 87.6)
- removed the G*** at (134.6, 53.3)
- removed the G*** at (71.1, 86.4)
- removed the G*** at (90.2, 71.1)
- removed the G*** at (218.4, 84.7)
- removed the G*** at (102.6, 85.3)
- removed the G*** at (57.1, 85.7)
- removed the G*** at (186.9, 82.2)
- removed the G*** at (160.0, 67.3)
- removed the G*** at (108.0, 58.4)
- removed the G*** at (241.6, 90.2)
- removed the G*** at (221.5, 47.6)
- removed the G*** at (61.5, 62.9)
- removed the G*** at (141.4, 82.4)
Routing:
- removed copper zone on B.Cu, net GND
- removed copper zone on F.Cu, net GND
Other:
- board text added: "Pro Micro here! Component side faces away from the PCB. Rev 2.0"
- board text removed: "CAUTION: Toxic Memes. DO NOT EAT. Do not wash with beer."
- board text removed: "CONTRA"
- board text removed: "Extremely low-cost Ortholinear keyboard"
- board text removed: "Pro Micro here! Component side faces away from the PCB. Rev 1.6"
- board text removed: "criminally cheap ortho"
